Commit message: mounted on robot

File: kortex_description/robots/gen3.xacro (robot description, xacro)
@@ -55,5 +55,5 @@
         use_external_cable="$(arg use_external_cable)"
         initial_positions="${xacro.load_yaml(initial_positions_file)}" >
-        <origin xyz="0 0 0" rpy="0 0 0" />  <!-- position robot in the world -->
+        <origin xyz="0 0 0" rpy="0 0.7853982 0" />  <!-- position robot in the world -->
     </xacro:load_robot>
 </robot>
