Commit message: scoop stl

File: kortex_description/arms/gen3/7dof/urdf/gen3_macro.xacro (robot description, xacro)
@@ -447,4 +447,33 @@
         xyz="0 0 0" />
     </joint>
+    <!-- Scoop Link -->
+    <link name="${prefix}spacer_scoop_link">
+      <visual>
+        <origin xyz="0 0 0" rpy="0 0 0" />
+        <geometry>
+          <mesh filename="file://$(find kortex_description)/arms/gen3/${dof}dof/meshes/spacer_scoop.stl" />
+        </geometry>
+        <material name="">
+          <color rgba="0.75294 0.75294 0.75294 1" />
+        </material>
+      </visual>
+      <collision>
+        <origin xyz="0 0 0" rpy="0 0 0" />
+        <geometry>
+          <mesh filename="file://$(find kortex_description)/arms/gen3/${dof}dof/meshes/spacer_scoop.stl" />
+        </geometry>
+      </collision>
+    </link>
+    <joint
+      name="${prefix}spacer_scoop_joint"
+      type="fixed">
+      <origin xyz="0 0 0" rpy="0 0 0" />
+      <parent
+        link="${prefix}end_effector_link" />
+      <child
+        link="${prefix}spacer_scoop_link" />
+      <axis
+        xyz="0 0 0" />
+    </joint>
     <xacro:if value="${vision}">
       <!-- sim camera needs to be rotated which might not apply to built in vision module -->

Commit message: no stl scoop for now

File: kortex_description/arms/gen3/7dof/urdf/gen3_macro.xacro (robot description, xacro)
@@ -448,18 +448,18 @@
     </joint>
     <!-- Scoop Link -->
-    <link name="${prefix}spacer_scoop_link">
-      <visual>
-        <origin xyz="0 0 0" rpy="0 0 0" />
-        <geometry>
-          <mesh filename="file://$(find kortex_description)/arms/gen3/${dof}dof/meshes/spacer_scoop.stl" />
-        </geometry>
-        <material name="">
-          <color rgba="0.75294 0.75294 0.75294 1" />
-        </material>
-      </visual>
-      <collision>
-        <origin xyz="0 0 0" rpy="0 0 0" />
-        <geometry>
-          <mesh filename="file://$(find kortex_description)/arms/gen3/${dof}dof/meshes/spacer_scoop.stl" />
+    <!-- <link name="${prefix}spacer_scoop_link">
+      <visual>
+        <origin xyz="0 0 0" rpy="0 0 0" />
+        <geometry>
+          <mesh filename="file://$(find kortex_description)/arms/gen3/${dof}dof/meshes/spacer_scoop.STL" scale="0.001 0.001 0.001"/>
+        </geometry>
+        <material name="">
+          <color rgba="0.75294 0.75294 0.75294 1" />
+        </material>
+      </visual>
+      <collision>
+        <origin xyz="0 0 0" rpy="0 0 0" />
+        <geometry>
+          <mesh filename="file://$(find kortex_description)/arms/gen3/${dof}dof/meshes/spacer_scoop.STL" />
         </geometry>
       </collision>
@@ -475,5 +475,5 @@
       <axis
         xyz="0 0 0" />
-    </joint>
+    </joint> -->
     <xacro:if value="${vision}">
       <!-- sim camera needs to be rotated which might not apply to built in vision module -->

Commit message: stl for scoop

File: kortex_description/arms/gen3/7dof/urdf/gen3_macro.xacro (robot description, xacro)
@@ -448,5 +448,5 @@
     </joint>
     <!-- Scoop Link -->
-    <!-- <link name="${prefix}spacer_scoop_link">
+    <link name="${prefix}spacer_scoop_link">
       <visual>
         <origin xyz="0 0 0" rpy="0 0 0" />
@@ -475,5 +475,5 @@
       <axis
         xyz="0 0 0" />
-    </joint> -->
+    </joint>
     <xacro:if value="${vision}">
       <!-- sim camera needs to be rotated which might not apply to built in vision module -->

Commit message: roation of scoop

File: kortex_description/arms/gen3/7dof/urdf/gen3_macro.xacro (robot description, xacro)
@@ -468,5 +468,5 @@
       name="${prefix}spacer_scoop_joint"
       type="fixed">
-      <origin xyz="0 0 0" rpy="0 0 0" />
+      <origin xyz="0 0 0" rpy="0 0 ${-PI}" />
       <parent
         link="${prefix}end_effector_link" />

Commit message: cartesian compliance and force

File: kortex_description/arms/gen3/7dof/urdf/gen3_macro.xacro (robot description, xacro)
@@ -447,6 +447,21 @@
         xyz="0 0 0" />
     </joint>
+    <link name="robot_mounting_link" />
+    <joint name="robot_mounting_joint" type="fixed">
+        <parent link="${prefix}end_effector_link" />
+        <child link = "robot_mounting_link" />
+        <origin xyz="0.0 0.0 0.0" rpy="0.0 0.0 0.0" />
+    </joint>
+    <xacro:arg name="bota_ft_sensor_link_name" default="bota_ft_sensor" />
+    <!-- SensONE GEN0 EtherCAT -->
+    <xacro:include filename="$(find bota_driver)/urdf/BFT_SENS_ECAT_M8.urdf.xacro" />
+    <xacro:BFT_SENS_ECAT_M8 prefix="$(arg bota_ft_sensor_link_name)" />
+    <joint name="robot_mounting_link_to_bota_ft_sensor" type="fixed">
+        <parent link="robot_mounting_link" />
+        <child link = "$(arg bota_ft_sensor_link_name)_mounting" />
+        <origin xyz="0.0 0.0 0.0" rpy="0.0 0.0 0.0" />
+    </joint>
     <!-- Scoop Link -->
-    <link name="${prefix}spacer_scoop_link">
+    <!-- <link name="${prefix}spacer_scoop_link">
       <visual>
         <origin xyz="0 0 0" rpy="0 0 0" />
@@ -475,5 +490,5 @@
       <axis
         xyz="0 0 0" />
-    </joint>
+    </joint> -->
     <xacro:if value="${vision}">
       <!-- sim camera needs to be rotated which might not apply to built in vision module -->

Commit message: bota sensor

File: kortex_description/arms/gen3/7dof/urdf/gen3_macro.xacro (robot description, xacro)
@@ -447,9 +447,34 @@
         xyz="0 0 0" />
     </joint>
+    <!-- Kinova to Bota adapt-->
+    <link name="kinova_bota_adapt_link" >
+      <visual>
+        <origin xyz="0 0 0" rpy="0 0 0" />
+        <geometry>
+          <mesh filename="file://$(find kortex_description)/arms/gen3/${dof}dof/meshes/kinova_bota_adapt.stl" scale="0.001 0.001 0.001"/>
+        </geometry>
+        <material name="">
+          <color rgba="0.75294 0.75294 0.75294 1" />
+        </material>
+      </visual>
+      <collision>
+        <origin xyz="0 0 0" rpy="0 0 0" />
+        <geometry>
+          <mesh filename="file://$(find kortex_description)/arms/gen3/${dof}dof/meshes/kinova_bota_adapt.stl" scale="0.001 0.001 0.001"/>
+        </geometry>
+      </collision>
+    </link>
+    <joint name="kinova_bota_adapt_joint" type="fixed">
+      <origin xyz="0 0 0" rpy="0 0 0" />
+      <parent link="${prefix}end_effector_link" />
+      <child link="kinova_bota_adapt_link" />
+      <axis xyz="0 0 0" />
+    </joint>
+    <!-- Bota sensor -->
     <link name="robot_mounting_link" />
     <joint name="robot_mounting_joint" type="fixed">
-        <parent link="${prefix}end_effector_link" />
+        <parent link="kinova_bota_adapt_link" />
         <child link = "robot_mounting_link" />
-        <origin xyz="0.0 0.0 0.0" rpy="0.0 0.0 0.0" />
+        <origin xyz="0.0 0.0 0.016" rpy="0.0 0.0 0.0" />
     </joint>
     <xacro:arg name="bota_ft_sensor_link_name" default="bota_ft_sensor" />
@@ -460,8 +485,32 @@
         <parent link="robot_mounting_link" />
         <child link = "$(arg bota_ft_sensor_link_name)_mounting" />
-        <origin xyz="0.0 0.0 0.0" rpy="0.0 0.0 0.0" />
+        <origin xyz="0 0 0" rpy="0.0 0.0 ${-PI}" />
+    </joint>
+    <!-- Bota to Scoop adapt -->
+    <link name="bota_scoop_adapt_link" >
+      <visual>
+        <origin xyz="0 0 0" rpy="0 0 0" />
+        <geometry>
+          <mesh filename="file://$(find kortex_description)/arms/gen3/${dof}dof/meshes/bota_scoop_adapt.stl" scale="0.001 0.001 0.001"/>
+        </geometry>
+        <material name="">
+          <color rgba="0.75294 0.75294 0.75294 1" />
+        </material>
+      </visual>
+      <collision>
+        <origin xyz="0 0 0" rpy="0 0 0" />
+        <geometry>
+          <mesh filename="file://$(find kortex_description)/arms/gen3/${dof}dof/meshes/bota_scoop_adapt.stl" scale="0.001 0.001 0.001"/>
+        </geometry>
+      </collision>
+    </link>
+    <joint name="bota_scoop_adapt_joint" type="fixed">
+      <origin xyz="0 0 0.035" rpy="0 0 0" />
+      <parent link="$(arg bota_ft_sensor_link_name)_mounting" />
+      <child link="bota_scoop_adapt_link" />
+      <axis xyz="0 0 0" />
     </joint>
     <!-- Scoop Link -->
-    <!-- <link name="${prefix}spacer_scoop_link">
+    <link name="${prefix}spacer_scoop_link">
       <visual>
         <origin xyz="0 0 0" rpy="0 0 0" />
@@ -480,15 +529,10 @@
       </collision>
     </link>
-    <joint
-      name="${prefix}spacer_scoop_joint"
-      type="fixed">
-      <origin xyz="0 0 0" rpy="0 0 ${-PI}" />
-      <parent
-        link="${prefix}end_effector_link" />
-      <child
-        link="${prefix}spacer_scoop_link" />
-      <axis
-        xyz="0 0 0" />
-    </joint> -->
+    <joint name="${prefix}spacer_scoop_joint" type="fixed">
+      <origin xyz="0 0 0.018" rpy="0 0 0" />
+      <parent link="bota_scoop_adapt_link" />
+      <child link="${prefix}spacer_scoop_link" />
+      <axis xyz="0 0 0" />
+    </joint>
     <xacro:if value="${vision}">
       <!-- sim camera needs to be rotated which might not apply to built in vision module -->

Commit message: bota sensor v2

File: kortex_description/arms/gen3/7dof/urdf/gen3_macro.xacro (robot description, xacro)
@@ -506,6 +506,6 @@
     </link>
     <joint name="bota_scoop_adapt_joint" type="fixed">
-      <origin xyz="0 0 0.035" rpy="0 0 0" />
-      <parent link="$(arg bota_ft_sensor_link_name)_mounting" />
+      <origin xyz="0 0 0" rpy="0 0 0" />
+      <parent link="$(arg bota_ft_sensor_link_name)_wrench" />
       <child link="bota_scoop_adapt_link" />
       <axis xyz="0 0 0" />

Commit message: removed bota from urdf

File: kortex_description/arms/gen3/7dof/urdf/gen3_macro.xacro (robot description, xacro)
@@ -448,5 +448,5 @@
     </joint>
     <!-- Kinova to Bota adapt-->
-    <link name="kinova_bota_adapt_link" >
+    <!-- <link name="kinova_bota_adapt_link" >
       <visual>
         <origin xyz="0 0 0" rpy="0 0 0" />
@@ -470,7 +470,7 @@
       <child link="kinova_bota_adapt_link" />
       <axis xyz="0 0 0" />
-    </joint>
+    </joint> -->
     <!-- Bota sensor -->
-    <link name="robot_mounting_link" />
+    <!-- <link name="robot_mounting_link" />
     <joint name="robot_mounting_joint" type="fixed">
         <parent link="kinova_bota_adapt_link" />
@@ -478,7 +478,7 @@
         <origin xyz="0.0 0.0 0.016" rpy="0.0 0.0 0.0" />
     </joint>
-    <xacro:arg name="bota_ft_sensor_link_name" default="bota_ft_sensor" />
+    <xacro:arg name="bota_ft_sensor_link_name" default="bota_ft_sensor" /> -->
     <!-- SensONE GEN0 EtherCAT -->
-    <xacro:include filename="file://$(find kinova_gen3n7)/bota_urdf/BFT_SENS_ECAT_M8.urdf.xacro" />
+    <!-- <xacro:include filename="$(find kinova_gen3n7)/bota_urdf/BFT_SENS_ECAT_M8.urdf.xacro" />
     <xacro:BFT_SENS_ECAT_M8 prefix="$(arg bota_ft_sensor_link_name)" />
     <joint name="robot_mounting_link_to_bota_ft_sensor" type="fixed">
@@ -486,7 +486,7 @@
         <child link = "$(arg bota_ft_sensor_link_name)_mounting" />
         <origin xyz="0 0 0" rpy="0.0 0.0 ${-PI}" />
-    </joint>
+    </joint> -->
     <!-- Bota to Scoop adapt -->
-    <link name="bota_scoop_adapt_link" >
+    <!-- <link name="bota_scoop_adapt_link" >
       <visual>
         <origin xyz="0 0 0" rpy="0 0 0" />
@@ -510,5 +510,5 @@
       <child link="bota_scoop_adapt_link" />
       <axis xyz="0 0 0" />
-    </joint>
+    </joint> -->
     <!-- Scoop Link -->
     <link name="${prefix}spacer_scoop_link">
@@ -530,6 +530,6 @@
     </link>
     <joint name="${prefix}spacer_scoop_joint" type="fixed">
-      <origin xyz="0 0 0.018" rpy="0 0 0" />
-      <parent link="bota_scoop_adapt_link" />
+      <origin xyz="0 0 0" rpy="0 0 ${-PI}" />
+      <parent link="${prefix}end_effector_link" />
       <child link="${prefix}spacer_scoop_link" />
       <axis xyz="0 0 0" />
